Commit message: 完美的Py模块化架构雏形！

File: mode/try2.SLDASM/urdf/try2.SLDASM.urdf (robot description, URDF)
Before this commit: robot try.SLDASM, 1 links, 0 joints
Links:
- link base_link: mass 0.000389416654106519 -> 0.138629348190767; geometry collision mesh filename=T:\Learn_More\learn from project\mujocu\try2.SLDASM\meshes\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; visual mesh filename=T:\Learn_More\learn from project\mujocu\try2.SLDASM\meshes\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
